File: hardware/shield_v01/wat.kicad_pcb (KiCad board)
At the start: 2 copper layers, 101.8 x 85.9 mm, 51 parts, among them P1 PINZA_1, P10 SCL-INT6, P102 CAUDAL_1, P103 V_IN, P106 18b20, P109 LCD_I2C, P11 SDA-INT5, P110 ARD_DI_06, P111 ARD_ALI_04, P2 PINZA_7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

Commit message: desrrollo pcb
Parts:
- R104: value 2K -> R18
- R9: value R18 -> 2K
- moved R9 111.3 mm to (151.1, 57.1), turned to 0 degrees
- moved W102 90.4 mm to (92.7, 62.2)
- moved C106 89.5 mm to (105.4, 67.3), turned to 180 degrees
- moved W101 80.3 mm to (185.4, 73.7)
- moved C105 80.0 mm to (181.6, 68.6), turned to 180 degrees
- moved C8 73.2 mm to (178.4, 118.1)
- moved P7 73.2 mm to (179.1, 124.5)
- moved P1 72.3 mm to (94.0, 125.7)
- moved C102 71.9 mm to (94.0, 119.4)
- moved R4 65.6 mm to (97.2, 119.4), turned to 90 degrees
- moved R10 65.6 mm to (182.2, 118.7), turned to 90 degrees
- moved P3 64.7 mm to (104.1, 125.7)
- moved P5 59.9 mm to (114.9, 125.7)
- moved R104 59.8 mm to (129.5, 118.7), turned to 90 degrees
- moved C4 59.0 mm to (102.9, 119.4)
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Connections:
- R1 pad 1: /Ves_3V3 -> /Vpc_5V
- R104 pad 1: /18b20 -> /Ref_medida
- R104 pad 2: /Vpc_5V -> /intensidad_4
- R9 pad 1: /Ref_medida -> /18b20
- R9 pad 2: /intensidad_4 -> /Vpc_5V

Commit message: desarrollo pcb v0
Parts:
- removed C102, C103: 100nF, Capacitors_ThroughHole:C_Disc_D3_P2.5
- removed R104: R18, Resistors_ThroughHole:Resistor_Horizontal_RM10mm
- removed U106: NANO, oscar_libreria_huellas:arduino_nano
- added C1: 100nF, Capacitors_ThroughHole:C_Disc_D3_P2.5, F.Cu at (94.6, 116.8)
- added C2: 100nF, Capacitors_ThroughHole:C_Disc_D3_P2.5, F.Cu at (151.8, 116.8)
- added R12: R18, Resistors_ThroughHole:Resistor_Horizontal_RM10mm, F.Cu at (129.0, 117.0)
- moved R1 46.6 mm to (142.2, 99.7)
- moved R3 41.3 mm to (146.1, 109.9)
- moved C101 39.1 mm to (135.9, 110.5), turned to 180 degrees
- moved P11 12.2 mm to (152.4, 80.0), turned to 270 degrees
- moved P10 12.1 mm to (152.4, 86.4), turned to 270 degrees
- moved P109 11.9 mm to (142.2, 78.1)
- moved R5 8.85 mm to (156.0, 117.0)
- moved P2 8.80 mm to (152.9, 123.6)
- moved R7 7.63 mm to (166.0, 117.0)
- moved P4 7.48 mm to (162.9, 123.6)
- moved C5 7.27 mm to (162.0, 117.0)
- moved C105 6.48 mm to (180.3, 62.2), turned to 90 degrees
- moved R11 6.08 mm to (176.0, 117.0)
- moved P8 5.96 mm to (172.9, 123.6)
- moved C9 5.74 mm to (172.0, 117.0)
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Routing:
- net /Ref_medida: track 0.00 -> 235.4 mm
- net /Var_8V: track 0.20 -> 208.4 mm, vias 0 -> 2
- net /Vpc_5V: track 0.00 -> 105.0 mm, vias 0 -> 4
- net /intensidad_8: track 0.00 -> 74.9 mm
- net /caudal_1: track 0.00 -> 71.9 mm
- net /intensidad_7: track 0.00 -> 68.0 mm
- net /intensidad_5: track 0.00 -> 67.2 mm
- net /18b20: track 0.00 -> 57.7 mm
- net /inten_5_SDA: track 0.00 -> 55.4 mm
- net /intensidad_6: track 0.00 -> 53.2 mm
- net /intensidad_4: track 0.00 -> 48.6 mm
- net /inten_6_SCL: track 0.00 -> 42.5 mm
- net /intensidad_3: track 0.00 -> 41.9 mm
- net /e_tx: track 0.00 -> 38.3 mm
- net /intensidad_2: track 0.00 -> 35.7 mm
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
Commit message: pcb simplificar a 6 medidas
Parts:
- removed C104, C108, C9: 100nF, Capacitors_ThroughHole:C_Disc_D3_P2.5
- removed P10: SCL-INT6, Pin_Headers:Pin_Header_Straight_1x03
- removed P11: SDA-INT5, Pin_Headers:Pin_Header_Straight_1x03
- removed P7: PINZA_5, Connect:bornier2
- removed P8: PINZA_6, Connect:bornier2
- removed R10, R11: R18, Resistors_ThroughHole:Resistor_Horizontal_RM10mm
- added C3: 100nF, Capacitors_THT:C_Disc_D5.0mm_W2.5mm_P5.00mm, F.Cu at (93.3, 54.6)
- C1, C2, C4, C5, C6, C7, C8: footprint Capacitors_ThroughHole:C_Disc_D3_P2.5 -> Capacitors_THT:C_Disc_D5.0mm_W2.5mm_P5.00mm
- moved C8 62.5 mm to (168.9, 55.9)
- moved R1 8.03 mm to (144.8, 92.1)
- moved C101 4.49 mm to (139.1, 107.3)
- moved C7 2.86 mm to (127.6, 118.1)
- moved R3 2.84 mm to (144.8, 107.3)
- moved R5 2.73 mm to (155.6, 114.3)
- moved R7 2.71 mm to (165.7, 114.3)
- moved C6 2.71 mm to (117.5, 118.1)
- moved R4 2.70 mm to (99.1, 114.3)
- moved R6 2.67 mm to (107.3, 114.9)
- moved C2 2.62 mm to (154.3, 117.5)
- moved C1 2.62 mm to (97.2, 117.5)
- moved C4 2.57 mm to (107.3, 118.1)
- moved R8 2.57 mm to (117.5, 114.9)
- moved C5 2.51 mm to (164.5, 117.5)
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Connections:
- C8 pad 1: /Ref_medida -> /caudal_1
- C8 pad 2: /intensidad_5 -> GND
- P9 pad 5: /inten_5_SDA -> /sda
- P9 pad 6: /inten_6_SCL -> /scl
Routing:
- net /intensidad_5: track 67.2 -> 0.00 mm
- net /inten_5_SDA: track 55.4 -> 0.00 mm
- net /intensidad_6: track 53.2 -> 0.00 mm
- net /inten_6_SCL: track 42.5 -> 0.00 mm
- net /sda: track 5.87 -> 42.9 mm
- net /scl: track 8.94 -> 38.0 mm
- net /Vpc_5V: track 105.0 -> 133.2 mm, vias 4 -> 2
- net /intensidad_4: track 48.6 -> 63.8 mm
- net /Ref_medida: track 235.4 -> 220.8 mm
- net /Ves_3V3: track 35.9 -> 44.5 mm
- net /caudal_1: track 71.9 -> 78.2 mm
- net /intensidad_2: track 35.7 -> 32.8 mm
- net /Var_8V: track 208.4 -> 205.7 mm, vias 2 -> 0
- net /intensidad_8: track 74.9 -> 77.3 mm
- net /intensidad_7: track 68.0 -> 70.4 mm
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