File: hardware/shield_v04/wat.kicad_pcb (KiCad board)
At the start: 2 copper layers, 101.8 x 85.9 mm, 49 parts, among them P1 PINZA_1, P102 CAUDAL_1, P103 V_IN, P106 18b20, P109 LCD_I2C, P110 ARD_DI_06, P111 ARD_ALI_04, P2 PINZA_7, P3 PINZA_2, P4 PINZA_8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

Commit message: pcb version con acs712
Parts:
- removed C8: 100nF, Capacitors_THT:C_Disc_D5.0mm_W2.5mm_P5.00mm
- removed D105: 1N4007, Diodes_ThroughHole:Diode_DO-35_SOD27_Horizontal_RM10
- removed P102: CAUDAL_1, Connect:bornier2
- removed P106: 18b20, Connect:bornier3
- removed R2: 10K, Resistors_ThroughHole:Resistor_Horizontal_RM10mm
- removed R9: 2K, Resistors_ThroughHole:Resistor_Horizontal_RM10mm
- added C1: 100nF, Capacitors_THT:C_Disc_D5.0mm_W2.5mm_P5.00mm, F.Cu at (150.4, 55.1)
- added C11: 100nF, Capacitors_THT:C_Disc_D5.0mm_W2.5mm_P5.00mm, F.Cu at (155.4, 117.9)
- C10: footprint Capacitors_ThroughHole:C_Disc_D3_P2.5 -> Capacitors_THT:C_Disc_D5.0mm_W2.5mm_P5.00mm
- moved P103 169.6 mm to (96.0, 123.7)
- moved U1 118.2 mm to (115.1, 119.1), turned to 0 degrees
- moved D104 100.7 mm to (93.5, 107.2), turned to 270 degrees
- moved C9 99.5 mm to (134.4, 116.6)
- moved W103 95.5 mm to (128.5, 123.7)
- moved C105 92.7 mm to (99.3, 107.2), turned to 270 degrees
- moved R4 84.8 mm to (169.9, 64.3), turned to 0 degrees
- moved C6 82.3 mm to (170.4, 55.1), turned to 0 degrees
- moved C7 82.1 mm to (180.3, 55.1), turned to 0 degrees
- moved C4 82.1 mm to (160.5, 55.1), turned to 0 degrees
- moved W101 79.4 mm to (107.2, 106.9)
- moved R12 68.7 mm to (181.1, 64.3), turned to 0 degrees
- moved R6 67.2 mm to (158.8, 64.3), turned to 0 degrees
- moved C10 62.6 mm to (165.4, 117.9), turned to 180 degrees
- moved P7 55.7 mm to (162.8, 123.7)
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