File: hardware/shield_v04/wat.sch (KiCad schematic (older format))
At the start: 52 parts, among them P1 PINZA_1, P102 CAUDAL_1, P103 V_IN, P106 18b20, P109 LCD_I2C, P110 ARD_DI_06, P111 ARD_ALI_04, P2 PINZA_7, P3 PINZA_2, P4 PINZA_8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

Commit message: pcb version con acs712
Parts:
- C1: footprint Capacitors_ThroughHole:C_Disc_D12_P7.75 -> Capacitors_THT:C_Disc_D5.0mm_W2.5mm_P5.00mm
- C10: footprint Capacitors_ThroughHole:C_Disc_D3_P2.5 -> Capacitors_THT:C_Disc_D5.0mm_W2.5mm_P5.00mm
- C11: footprint Capacitors_ThroughHole:C_Disc_D6_P5 -> Capacitors_THT:C_Disc_D5.0mm_W2.5mm_P5.00mm
Changed lines of the file:
@@
 LIBS:mp-1584
 LIBS:nano
+LIBS:current_sensor-cache
 LIBS:wat-cache
 EELAYER 25 0
@@
 F 0 "C1" H 2435 6005 50  0000 L CNN
 F 1 "100nF" H 2435 5805 50  0000 L CNN
-F 2 "Capacitors_ThroughHole:C_Disc_D12_P7.75" H 2448 5755 50  0001 C CNN
+F 2 "Capacitors_THT:C_Disc_D5.0mm_W2.5mm_P5.00mm" H 2448 5755 50  0001 C CNN
 F 3 "" H 2410 5905 50  0000 C CNN
 	1    2410 5905
@@
 F 0 "C11" H 9790 5910 50  0000 L CNN
 F 1 "100nF" H 9790 5710 50  0000 L CNN
-F 2 "Capacitors_ThroughHole:C_Disc_D6_P5" H 9803 5660 50  0001 C CNN
+F 2 "Capacitors_THT:C_Disc_D5.0mm_W2.5mm_P5.00mm" H 9803 5660 50  0001 C CNN
 F 3 "" H 9765 5810 50  0000 C CNN
 	1    9765 5810
@@
 F 0 "C10" H 1640 7120 50  0000 L CNN
 F 1 "100nF" H 1640 6920 50  0000 L CNN
-F 2 "Capacitors_ThroughHole:C_Disc_D3_P2.5" H 1653 6870 50  0001 C CNN
+F 2 "Capacitors_THT:C_Disc_D5.0mm_W2.5mm_P5.00mm" H 1653 6870 50  0001 C CNN
 F 3 "" H 1615 7020 50  0000 C CNN
 	1    1615 7020
